File: UDB.kicad_pcb (KiCad board)
At the start: 4 copper layers, 18 x 16.5 mm, 14 parts, among them J1 TYPE-C-31-M12_13, J2 SM04B-SRSS-TB(LF)(SN), U1 TPD4E05U06DQAR

Commit message: Densus Logo version
Parts:
- removed G1: Unified-Daughterboard-Logo, Unified-Daughterboard-Logo:Unified-Daughterboard-Logo.pretty
- added G***: LOGO, LOGO, B.Cu at (75.0, 68.4)
